File: PCB/clackintosh-jr.kicad_pcb (KiCad board)
At the start: 2 copper layers, 81.1 x 65.8 mm, 30 parts, among them J1 Conn_01x04_Pin, SW1 SW_Push, SW2 SW_Push, SW3 SW_Push, SW4 SW_Push, SW5 SW_Push, SW6 SW_Push, SW7 SW_Push, SW8 SW_Push, SW9 RotaryEncoder_Switch_MP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

Commit message: update readme + production folder
Parts:
- moved D10 0.55 mm to (181.2, 126.5)
- moved D12 0.44 mm to (181.5, 106.8)
Routing:
- net +5V: track 194.2 -> 195.8 mm
Changed lines of the file:
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@@
 			(outputformat 1)
 			(mirror no)
-			(drillshape 1)
+			(drillshape 0)
 			(scaleselection 1)
-			(outputdirectory "")
+			(outputdirectory "prod/")
 		)
 	)
@@
 	(footprint "LED:SK6812-MINI-E"
 		(layer "B.Cu")
-		(at 181.725 126.49 180)
+		(at 181.175 126.49 180)
 		(property "Reference" "D10"
 			(at 0 -2.1 0)
@@
 	(footprint "LED:SK6812-MINI-E"
 		(layer "B.Cu")
-		(at 181.9 106.74 180)
+		(at 181.475 106.85 180)
 		(property "Reference" "D12"
 			(at 0 -2.1 0)
@@
 	)
 	(segment
-		(start 187.5045 98.1918)
-		(end 187.7658 98.4531)
+		(start 178.9683 120.8317)
+		(end 178.4 121.4)
 		(width 0.2)
 		(layer "B.Cu")
@@
 	)
 	(segment
-		(start 178.9683 120.826)
-		(end 178.9683 125.6583)
+		(start 187.5045 98.1918)
+		(end 187.7658 98.4531)
 		(width 0.2)
 		(layer "B.Cu")
@@
 	)
 	(segment
+		(start 178.5 121.5)
+		(end 178.5 125.74)
+		(width 0.2)
+		(layer "B.Cu")
+		(net 13)
+	)
+	(segment
 		(start 189.185 71.1185)
 		(end 190.02 71.1185)
@@
 	)
 	(segment
+		(start 178.4 121.4)
+		(end 178.5 121.5)
+		(width 0.2)
+		(layer "B.Cu")
+		(net 13)
+	)
+	(segment
 		(start 187.7658 114.8858)
 		(end 184.5419 118.1097)
@@
 	)
 	(segment
+		(start 178.9683 120.826)
+		(end 178.9683 120.8317)
+		(width 0.2)
+		(layer "B.Cu")
+		(net 13)
+	)
+	(segment
 		(start 178.9683 125.6583)
 		(end 179.05 125.74)
@@
 	)
 	(segment
+		(start 178.3 108.1)
+		(end 178.3 108.7)
+		(width 0.2)
+		(layer "B.Cu")
+		(net 14)
+	)
+	(segment
 		(start 121.625 127.49)
 		(end 121.1117 127.49)
@@
 	)
 	(segment
+		(start 178.3 108.7)
+		(end 178.1983 108.8017)
+		(width 0.2)
+		(layer "B.Cu")
+		(net 14)
+	)
+	(segment
 		(start 147.8542 126.3516)
 		(end 147.8542 128.4463)
@@
 	)
 	(segment
-		(start 178.1983 115.6172)
-		(end 178.1983 107.49)
-		(width 0.2)
-		(layer "B.Cu")
-		(net 14)
-	)
-	(segment
 		(start 147.8542 128.4463)
 		(end 147.4663 128.8342)
@@
 	)
 	(segment
-		(start 178.0069 127.2236)
+		(start 177.01525 128.21525)
 		(end 176.6303 128.6002)
 		(width 0.2)
@@
 	)
 	(segment
+		(start 178.8 107.6)
+		(end 178.3 108.1)
+		(width 0.2)
+		(layer "B.Cu")
+		(net 14)
+	)
+	(segment
 		(start 118.0289 124.9206)
 		(end 120.5983 127.49)
@@
 	)
 	(segment
+		(start 178.9683 116.3872)
+		(end 178.9683 120.221)
+		(width 0.2)
+		(layer "B.Cu")
+		(net 14)
+	)
+	(segment
 		(start 118.0289 110.1594)
 		(end 118.0289 124.9206)
@@
 	)
 	(segment
+		(start 177.474 127.7565)
+		(end 177.01525 128.21525)
+		(width 0.2)
+		(layer "B.Cu")
+		(net 14)
+	)
+	(segment
+		(start 178.1983 108.8017)
+		(end 178.1983 115.6172)
+		(width 0.2)
+		(layer "B.Cu")
+		(net 14)
+	)
+	(segment
+		(start 178.1983 115.6172)
+		(end 178.9683 116.3872)
+		(width 0.2)
+		(layer "B.Cu")
+		(net 14)
+	)
+	(segment
 		(start 178.0069 127.2236)
-		(end 178.0069 121.1824)
+		(end 177.01525 128.21525)
 		(width 0.2)
 		(layer "B.Cu")
@@
 	)
 	(segment
+		(start 178.9683 120.221)
+		(end 177.474 121.7153)
+		(width 0.2)
+		(layer "B.Cu")
+		(net 14)
+	)
+	(segment
 		(start 160.1298 101.3875)
 		(end 158.6471 102.8702)
@@
 	)
 	(segment
-		(start 178.9683 116.3872)
-		(end 178.1983 115.6172)
-		(width 0.2)
-		(layer "B.Cu")
-		(net 14)
-	)
-	(segment
 		(start 138.5697 128.5936)
 		(end 139.6733 127.49)
@@
 	)
 	(segment
-		(start 178.9683 120.221)
-		(end 178.9683 116.3872)
-		(width 0.2)
-		(layer "B.Cu")
-		(net 14)
-	)
-	(segment
-		(start 178.0069 121.1824)
-		(end 178.9683 120.221)
+		(start 173.945 71.1185)
+		(end 173.11 71.1185)
 		(width 0.2)
 		(layer "B.Cu")
@@
 	)
 	(segment
-		(start 173.945 71.1185)
-		(end 173.11 71.1185)
+		(start 177.474 121.7153)
+		(end 177.474 127.7565)
 		(width 0.2)
 		(layer "B.Cu")
@@
 	)
 	(segment
-		(start 139.6939 109.0886)
-		(end 139.6939 110.0058)
+		(start 184.0641 124.0896)
+		(end 184.0641 125.5259)
 		(width 0.2)
 		(layer "B.Cu")
@@
 	)
 	(segment
-		(start 184.575 104.6217)
-		(end 184.575 105.99)
+		(start 139.6939 109.0886)
+		(end 139.6939 110.0058)
 		(width 0.2)
 		(layer "B.Cu")
@@
 	)
 	(segment
-		(start 184.4 124.4255)
-		(end 184.4 125.74)
-		(width 0.2)
-		(layer "B.Cu")
-		(net 15)
-	)
-	(segment
 		(start 129.9983 87.3717)
 		(end 129.9983 86.07)
@@
 	)
 	(segment
+		(start 184.0641 125.5259)
+		(end 183.85 125.74)
+		(width 0.2)
+		(layer "B.Cu")
+		(net 15)
+	)
+	(segment
 		(start 147.1017 104.08)
 		(end 147.1017 106.49)
@@
 	)
 	(segment
+		(start 184.4438 105.8062)
+		(end 184.15 106.1)
+		(width 0.2)
+		(layer "B.Cu")
+		(net 15)
+	)
+	(segment
 		(start 126.975 120.9449)
 		(end 125.493 119.4629)
@@
 	)
 	(segment
-		(start 184.0641 124.0896)
-		(end 184.4 124.4255)
+		(start 184.4438 104.4905)
+		(end 184.4438 105.8062)
 		(width 0.2)
 		(layer "B.Cu")
@@
 	)
 	(segment
-		(start 176.1293 108.9806)
-		(end 179.1199 105.99)
+		(start 176.1293 108.5337)
+		(end 178.563 106.1)
 		(width 0.2)
 		(layer "B.Cu")
@@
 	(segment
 		(start 176.1293 117.3546)
-		(end 176.1293 108.9806)
+		(end 176.1293 108.5337)
 		(width 0.2)
 		(layer "B.Cu")
@@
 	)
 	(segment
-		(start 185.4267 124.3415)
-		(end 184.8398 123.7546)
+		(start 185.4267 127.24)
+		(end 183.85 127.24)
+		(width 0.2)
+		(layer "B.Cu")
+		(net 16)
+	)
+	(segment
+		(start 178.563 106.1)
+		(end 178.8 106.1)
 		(width 0.2)
 		(layer "B.Cu")
@@
 	)
 	(segment
-		(start 184.4 127.24)
-		(end 185.4267 127.24)
+		(start 185.4267 124.3415)
+		(end 184.8398 123.7546)
 		(width 0.2)
 		(layer "B.Cu")
@@
 	)
 	(segment
+		(start 179.7764 110.787)
+		(end 182.013 110.787)
+		(width 0.2)
+		(layer "B.Cu")
+		(net 19)
+	)
+	(segment
 		(start 139.6983 108.525)
 		(end 139.875 108.7017)
@@
 	)
 	(segment
-		(start 184.575 107.7875)
-		(end 181.5755 110.787)
+		(start 182.013 110.787)
+		(end 184.15 108.65)
 		(width 0.2)
 		(layer "B.Cu")
@@
 	)
 	(segment
-		(start 181.5755 110.787)
-		(end 179.7764 110.787)
+		(start 184.15 108.65)
+		(end 184.15 107.6)
 		(width 0.2)
 		(layer "B.Cu")
